Commit message: Fix joint names

File: manipulator_description/urdf/manipulator_h.xacro (robot description, xacro)
@@ -7,10 +7,10 @@
   <xacro:macro name="manipulator_h_robot" params="prefix joint_limited">
     <!-- Used for fixing robot to Gazebo 'link 1' -->
-    <link name="${prefix}base_link" >
+    <!-- <link name="${prefix}base_link" >
     </link>
     <joint name="shoulder_pan_joint" type="fixed">
       <parent link="${prefix}base_link"/>
-      <child link="${prefix}link1"/>
-    </joint>
+      <child link="${prefix}shoulder_link"/>
+    </joint> -->
     <!-- link 1 -->
     <link name="${prefix}shoulder_link">
@@ -38,5 +38,5 @@
     </link>
     <!-- Joint 1 -->
-    <joint name="${prefix}shoulder_lift_joint" type="revolute">
+    <joint name="${prefix}shoulder_pan_joint" type="revolute">
       <parent link="${prefix}shoulder_link" />
       <child link = "${prefix}upper_arm_link" />
@@ -71,5 +71,5 @@
     </link>
     <!-- Joint 2 -->
-    <joint name="${prefix}elbow_joint" type="revolute">
+    <joint name="${prefix}shoulder_lift_joint" type="revolute">
       <parent link="${prefix}upper_arm_link" />
       <child link = "${prefix}forearm_link" />
@@ -104,5 +104,5 @@
     </link>
     <!-- Joint 3 -->
-    <joint name="${prefix}wrist_1_joint" type="revolute">
+    <joint name="${prefix}elbow_joint" type="revolute">
       <parent link="${prefix}forearm_link" />
       <child link = "${prefix}wrist_1_link" />
@@ -137,5 +137,5 @@
     </link>
     <!-- Joint 4 -->
-    <joint name="${prefix}wrist_2_joint" type="revolute">
+    <joint name="${prefix}wrist_1_joint" type="revolute">
       <parent link="${prefix}wrist_1_link" />
       <child link = "${prefix}wrist_2_link" />
@@ -170,5 +170,5 @@
     </link>
     <!-- Joint 5 -->
-    <joint name="${prefix}wrist_3_joint" type="revolute">
+    <joint name="${prefix}wrist_2_joint" type="revolute">
       <parent link="${prefix}wrist_2_link" />
       <child link = "${prefix}wrist_3_link" />
@@ -203,5 +203,5 @@
     </link>
     <!-- Joint 6 -->
-    <joint name="${prefix}ee_fixed_joint" type="fixed">
+    <joint name="${prefix}wrist_3_joint" type="revolute">
       <parent link="${prefix}wrist_3_link" />
       <child link = "${prefix}ee_link" />

File: manipulator_description/urdf/manipulator_h_robot.xacro (robot description, xacro)
@@ -11,5 +11,5 @@
   <joint name="world_joint" type="fixed">
     <parent link="world" />
-    <child link = "base_link" />
+    <child link = "shoulder_link" />
     <origin xyz="0.0 0.0 0.0" rpy="0.0 0.0 0.0" />
   </joint>

Commit message: Allow passing parent link

File: manipulator_description/urdf/manipulator_h.xacro (robot description, xacro)
@@ -5,5 +5,5 @@
   <xacro:include filename="$(find manipulator_description)/urdf/materials.xacro" />
   <xacro:property name="pi" value="3.141592654" />
-  <xacro:macro name="manipulator_h_robot" params="prefix joint_limited">
+  <xacro:macro name="manipulator_h_robot" params="prefix joint_limited parent *origin">
     <!-- Used for fixing robot to Gazebo 'link 1' -->
     <!-- <link name="${prefix}base_link" >
@@ -13,4 +13,10 @@
       <child link="${prefix}shoulder_link"/>
     </joint> -->
+    <!-- First element of the arm fixed to the parent -->
+    <joint name="${parent}_${prefix}_base_joint" type="fixed">
+      <insert_block name="origin" />
+      <parent link="${parent}" />
+      <child link="${prefix}shoulder_link" />
+    </joint>
     <!-- link 1 -->
     <link name="${prefix}shoulder_link">

File: manipulator_description/urdf/manipulator_h_robot.xacro (robot description, xacro)
@@ -6,11 +6,8 @@
   <!-- manipulator -->
   <xacro:include filename="$(find manipulator_description)/urdf/manipulator_h.xacro" />
+  <link name="world" />
   <!-- arm -->
-  <xacro:manipulator_h_robot prefix="" joint_limited="false"/>
-  <link name="world" />
-  <joint name="world_joint" type="fixed">
-    <parent link="world" />
-    <child link="shoulder_link" />
-    <origin xyz="0.0 0.0 0.0" rpy="0.0 0.0 0.0" />
-  </joint>
+  <xacro:manipulator_h_robot prefix="" parent="world" joint_limited="false">
+    <origin xyz="0 0 0" rpy="0 0 0" />
+  </xacro:manipulator_h_robot>
 </robot>

Commit message: Move gazebo import lower in the hierarchy

File: manipulator_description/urdf/manipulator_h.xacro (robot description, xacro)
@@ -5,12 +5,7 @@
   <xacro:include filename="$(find manipulator_description)/urdf/materials.xacro" />
   <xacro:property name="pi" value="3.141592654" />
+  <!-- gazebo related stuff -->
+  <xacro:include filename="$(find manipulator_description)/urdf/common.xacro" />
   <xacro:macro name="manipulator_h_robot" params="prefix joint_limited parent *origin">
-    <!-- Used for fixing robot to Gazebo 'link 1' -->
-    <!-- <link name="${prefix}base_link" >
-    </link>
-    <joint name="shoulder_pan_joint" type="fixed">
-      <parent link="${prefix}base_link"/>
-      <child link="${prefix}shoulder_link"/>
-    </joint> -->
     <!-- First element of the arm fixed to the parent -->
     <joint name="${parent}_${prefix}_base_joint" type="fixed">

File: manipulator_description/urdf/manipulator_h_robot.xacro (robot description, xacro)
@@ -2,6 +2,4 @@
 <robot xmlns:xacro="http://www.ros.org/wiki/xacro"
        name="manipulator_h" >
-  <!-- common stuff -->
-  <xacro:include filename="$(find manipulator_description)/urdf/common.xacro" />
   <!-- manipulator -->
   <xacro:include filename="$(find manipulator_description)/urdf/manipulator_h.xacro" />

Commit message: Rename manipulator_h_robot to manipulator_h_arm

File: manipulator_description/urdf/manipulator_h.xacro (robot description, xacro)
@@ -7,5 +7,5 @@
   <!-- gazebo related stuff -->
   <xacro:include filename="$(find manipulator_description)/urdf/common.xacro" />
-  <xacro:macro name="manipulator_h_robot" params="prefix joint_limited parent *origin">
+  <xacro:macro name="manipulator_h_arm" params="prefix joint_limited parent *origin">
     <!-- First element of the arm fixed to the parent -->
     <joint name="${parent}_${prefix}_base_joint" type="fixed">

File: manipulator_description/urdf/manipulator_h_arm.xacro (robot description, xacro)
@@ -6,6 +6,6 @@
   <link name="world" />
   <!-- arm -->
-  <xacro:manipulator_h_robot prefix="" parent="world" joint_limited="false">
+  <xacro:manipulator_h_arm prefix="" parent="world" joint_limited="false">
     <origin xyz="0 0 0" rpy="0 0 0" />
-  </xacro:manipulator_h_robot>
+  </xacro:manipulator_h_arm>
 </robot>

Commit message: User prefixval for urdf

File: manipulator_description/urdf/manipulator_h.xacro (robot description, xacro)
@@ -5,15 +5,21 @@
   <xacro:include filename="$(find manipulator_description)/urdf/materials.xacro" />
   <xacro:property name="pi" value="3.141592654" />
+  <xacro:property name="prefix_val" value="" />
   <!-- gazebo related stuff -->
   <xacro:include filename="$(find manipulator_description)/urdf/common.xacro" />
   <xacro:macro name="manipulator_h_arm" params="prefix joint_limited parent *origin">
+    <!-- Suffix prefix with underscore -->
+    <xacro:if value="${prefix.__len__()}">
+      <xacro:property name="prefix_val" value="${prefix + '_'}" />
+    </xacro:if>
+    <xacro:manipulator_arm_gazebo prefix="${prefix}" prefix_val="${prefix_val}" />
     <!-- First element of the arm fixed to the parent -->
-    <joint name="${parent}_${prefix}_base_joint" type="fixed">
+    <joint name="${parent}_${prefix_val}_base_joint" type="fixed">
       <xacro:insert_block name="origin" />
       <parent link="${parent}" />
-      <child link="${prefix}shoulder_link" />
+      <child link="${prefix_val}shoulder_link" />
     </joint>
     <!-- link 1 -->
-    <link name="${prefix}shoulder_link">
+    <link name="${prefix_val}shoulder_link">
       <collision>
         <origin xyz="0 0 0.063" rpy="0 0 ${pi}"/>
@@ -39,7 +45,7 @@
     </link>
     <!-- Joint 1 -->
-    <joint name="${prefix}shoulder_pan_joint" type="revolute">
-      <parent link="${prefix}shoulder_link" />
-      <child link = "${prefix}upper_arm_link" />
+    <joint name="${prefix_val}shoulder_pan_joint" type="revolute">
+      <parent link="${prefix_val}shoulder_link" />
+      <child link = "${prefix_val}upper_arm_link" />
       <origin xyz="0 0 0.126" rpy="0 0 0"/>
       <axis xyz="0 0 1"/>
@@ -48,5 +54,5 @@
     </joint>
     <!-- link 2 -->
-    <link name="${prefix}upper_arm_link">
+    <link name="${prefix_val}upper_arm_link">
       <collision>
         <origin xyz="0 0 0.033" rpy="0 0 ${pi}"/>
@@ -72,7 +78,7 @@
     </link>
     <!-- Joint 2 -->
-    <joint name="${prefix}shoulder_lift_joint" type="revolute">
-      <parent link="${prefix}upper_arm_link" />
-      <child link = "${prefix}forearm_link" />
+    <joint name="${prefix_val}shoulder_lift_joint" type="revolute">
+      <parent link="${prefix_val}upper_arm_link" />
+      <child link = "${prefix_val}forearm_link" />
       <origin xyz="0 0 0.033" rpy="0 0 0"/>
       <axis xyz="0 1 0"/>
@@ -81,5 +87,5 @@
     </joint>
     <!-- link 3 -->
-    <link name="${prefix}forearm_link">
+    <link name="${prefix_val}forearm_link">
       <collision>
         <origin xyz="0.02 0 0.15" rpy="0 0 ${pi}"/>
@@ -105,7 +111,7 @@
     </link>
     <!-- Joint 3 -->
-    <joint name="${prefix}elbow_joint" type="revolute">
-      <parent link="${prefix}forearm_link" />
-      <child link = "${prefix}wrist_1_link" />
+    <joint name="${prefix_val}elbow_joint" type="revolute">
+      <parent link="${prefix_val}forearm_link" />
+      <child link = "${prefix_val}wrist_1_link" />
       <origin xyz="0.03 0.0 0.264" rpy="0 ${45.0*pi/180.0} 0" />
       <axis xyz="0 1 0"/>
@@ -114,5 +120,5 @@
     </joint>
     <!-- link 4 -->
-    <link name="${prefix}wrist_1_link">
+    <link name="${prefix_val}wrist_1_link">
       <collision>
         <origin xyz="-0.01 0.0 0.1" rpy="0 0 ${pi}" />
@@ -138,7 +144,7 @@
     </link>
     <!-- Joint 4 -->
-    <joint name="${prefix}wrist_1_joint" type="revolute">
-      <parent link="${prefix}wrist_1_link" />
-      <child link = "${prefix}wrist_2_link" />
+    <joint name="${prefix_val}wrist_1_joint" type="revolute">
+      <parent link="${prefix_val}wrist_1_link" />
+      <child link = "${prefix_val}wrist_2_link" />
       <origin xyz="-0.03 0.0 0.231" rpy="0 0 0" />
       <axis xyz="0 0 1" />
@@ -147,5 +153,5 @@
     </joint>
     <!-- link 5 -->
-    <link name="${prefix}wrist_2_link">
+    <link name="${prefix_val}wrist_2_link">
       <collision>
         <origin xyz="0.0 0.0 0.03" rpy="0 0 ${pi}" />
@@ -171,7 +177,7 @@
     </link>
     <!-- Joint 5 -->
-    <joint name="${prefix}wrist_2_joint" type="revolute">
-      <parent link="${prefix}wrist_2_link" />
-      <child link = "${prefix}wrist_3_link" />
+    <joint name="${prefix_val}wrist_2_joint" type="revolute">
+      <parent link="${prefix_val}wrist_2_link" />
+      <child link = "${prefix_val}wrist_3_link" />
       <origin xyz="0.0 0.0 0.027" rpy="0 0 0" />
       <axis xyz="0 1 0" />
@@ -180,5 +186,5 @@
     </joint>
     <!-- link 6 -->
-    <link name="${prefix}wrist_3_link">
+    <link name="${prefix_val}wrist_3_link">
       <collision>
         <origin xyz="0.0 0.0 0.08" rpy="0 0 ${pi}" />
@@ -204,7 +210,7 @@
     </link>
     <!-- Joint 6 -->
-    <joint name="${prefix}wrist_3_joint" type="revolute">
-      <parent link="${prefix}wrist_3_link" />
-      <child link = "${prefix}ee_link" />
+    <joint name="${prefix_val}wrist_3_joint" type="revolute">
+      <parent link="${prefix_val}wrist_3_link" />
+      <child link = "${prefix_val}ee_link" />
       <origin xyz="0.0 0.0 0.123" rpy="0 0 0" />
       <axis xyz="0 0 1" />
@@ -213,5 +219,5 @@
     </joint>
     <!-- End Effector -->
-    <link name="${prefix}ee_link">
+    <link name="${prefix_val}ee_link">
       <collision>
         <origin xyz="0.0 0.0 0.0" rpy="0 0 0" />
@@ -236,5 +242,5 @@
       </inertial>
     </link>
-    <xacro:manipulator_arm_transmission prefix="${prefix}" />
+    <xacro:manipulator_arm_transmission prefix="${prefix_val}" />
   </xacro:macro>
 </robot>

Commit message: Change the joint limits

File: manipulator_description/urdf/manipulator_h.xacro (robot description, xacro)
@@ -47,5 +47,5 @@
       <origin xyz="0 0 0.126" rpy="0 0 0"/>
       <axis xyz="0 0 1"/>
-      <limit velocity="6.5" effort="1000" lower="${-pi*0.6}" upper="${pi*0.6}" />
+      <limit velocity="6.5" effort="1000" lower="${-pi*0.95}" upper="${pi*0.95}" />
       <dynamics damping="0.7"/>
     </joint>
@@ -80,5 +80,5 @@
       <origin xyz="0 0 0.033" rpy="0 0 0"/>
       <axis xyz="0 1 0"/>
-      <limit velocity="6.5" effort="1000" lower="${-pi*0.45}" upper="${pi*0.45}" />
+      <limit velocity="6.5" effort="1000" lower="${-pi*0.6}" upper="${pi*0.6}" />
       <dynamics damping="0.7"/>
     </joint>
@@ -113,5 +113,5 @@
       <origin xyz="0.03 0.0 0.264" rpy="0 ${45.0*pi/180.0} 0" />
       <axis xyz="0 1 0"/>
-      <limit velocity="6.5" effort="1000" lower="${-pi*0.4}" upper="${pi*0.7}" />
+      <limit velocity="6.5" effort="1000" lower="${-pi*0.4}" upper="${pi*0.72}" />
       <dynamics damping="0.7"/>
     </joint>
@@ -146,5 +146,5 @@
       <origin xyz="-0.03 0.0 0.231" rpy="0 0 0" />
       <axis xyz="0 0 1" />
-      <limit velocity="6.5" effort="1000" lower="${-pi*0.6}" upper="${pi*0.6}" />
+      <limit velocity="6.5" effort="1000" lower="${-pi}" upper="${pi}" />
       <dynamics damping="0.7"/>
     </joint>
@@ -179,5 +179,5 @@
       <origin xyz="0.0 0.0 0.027" rpy="0 0 0" />
       <axis xyz="0 1 0" />
-      <limit velocity="6.5" effort="1000" lower="${-pi*0.45}" upper="${pi*0.45}" />
+      <limit velocity="6.5" effort="1000" lower="${-pi*0.5}" upper="${pi*0.5}" />
       <dynamics damping="0.7"/>
     </joint>
@@ -212,5 +212,5 @@
       <origin xyz="0.0 0.0 0.123" rpy="0 0 0" />
       <axis xyz="0 0 1" />
-      <limit velocity="6.5" effort="1000" lower="${-pi*0.6}" upper="${pi*0.6}" />
+      <limit velocity="6.5" effort="1000" lower="${-pi}" upper="${pi}" />
       <dynamics damping="0.7"/>
     </joint>

Commit message: Fix formatting

File: manipulator_description/urdf/manipulator_h.xacro (robot description, xacro)
@@ -22,5 +22,5 @@
         <origin xyz="0 0 0.063" rpy="0 0 ${pi}"/>
         <geometry>
-      <box size="0.06 0.06 0.126"/>
+          <box size="0.06 0.06 0.126"/>
         </geometry>
       </collision>
@@ -36,7 +36,7 @@
         <mass value="0.936"/>
         <inertia
-        ixx="1.0" ixy="0.0" ixz="0.0"
-        iyy="1.0" iyz="0.0"
-        izz="1.0"/>
+          ixx="1.0" ixy="0.0" ixz="0.0"
+          iyy="1.0" iyz="0.0"
+          izz="1.0"/>
       </inertial>
     </link>
@@ -44,5 +44,5 @@
     <joint name="${prefix_val}shoulder_pan_joint" type="revolute">
       <parent link="${prefix_val}shoulder_link" />
-      <child link = "${prefix_val}upper_arm_link" />
+      <child link="${prefix_val}upper_arm_link" />
       <origin xyz="0 0 0.126" rpy="0 0 0"/>
       <axis xyz="0 0 1"/>
@@ -55,5 +55,5 @@
         <origin xyz="0 0 0.033" rpy="0 0 ${pi}"/>
         <geometry>
-      <box size="0.07 0.15 0.08"/>
+          <box size="0.07 0.15 0.08"/>
         </geometry>
       </collision>
@@ -69,7 +69,7 @@
         <mass value="1.030"/>
         <inertia
-        ixx="1.0" ixy="0.0" ixz="0.0"
-        iyy="1.0" iyz="0.0"
-        izz="1.0"/>
+          ixx="1.0" ixy="0.0" ixz="0.0"
+          iyy="1.0" iyz="0.0"
+          izz="1.0"/>
       </inertial>
     </link>
@@ -77,5 +77,5 @@
     <joint name="${prefix_val}shoulder_lift_joint" type="revolute">
       <parent link="${prefix_val}upper_arm_link" />
-      <child link = "${prefix_val}forearm_link" />
+      <child link="${prefix_val}forearm_link" />
       <origin xyz="0 0 0.033" rpy="0 0 0"/>
       <axis xyz="0 1 0"/>
@@ -88,5 +88,5 @@
         <origin xyz="0.02 0 0.15" rpy="0 0 ${pi}"/>
         <geometry>
-      <box size="0.1 0.15 0.25"/>
+          <box size="0.1 0.15 0.25"/>
         </geometry>
       </collision>
@@ -102,7 +102,7 @@
         <mass value="1.404"/>
         <inertia
-        ixx="1.0" ixy="0.0" ixz="0.0"
-        iyy="1.0" iyz="0.0"
-        izz="1.0"/>
+          ixx="1.0" ixy="0.0" ixz="0.0"
+          iyy="1.0" iyz="0.0"
+          izz="1.0"/>
       </inertial>
     </link>
@@ -110,5 +110,5 @@
     <joint name="${prefix_val}elbow_joint" type="revolute">
       <parent link="${prefix_val}forearm_link" />
-      <child link = "${prefix_val}wrist_1_link" />
+      <child link="${prefix_val}wrist_1_link" />
       <origin xyz="0.03 0.0 0.264" rpy="0 ${45.0*pi/180.0} 0" />
       <axis xyz="0 1 0"/>
@@ -121,5 +121,5 @@
         <origin xyz="-0.01 0.0 0.1" rpy="0 0 ${pi}" />
         <geometry>
-      <box size="0.1 0.15 0.25" />
+          <box size="0.1 0.15 0.25" />
         </geometry>
       </collision>
@@ -135,7 +135,7 @@
         <mass value="1.236" />
         <inertia
-        ixx="1.0" ixy="0.0" ixz="0.0"
-        iyy="1.0" iyz="0.0"
-        izz="1.0"/>
+          ixx="1.0" ixy="0.0" ixz="0.0"
+          iyy="1.0" iyz="0.0"
+          izz="1.0"/>
       </inertial>
     </link>
@@ -143,5 +143,5 @@
     <joint name="${prefix_val}wrist_1_joint" type="revolute">
       <parent link="${prefix_val}wrist_1_link" />
-      <child link = "${prefix_val}wrist_2_link" />
+      <child link="${prefix_val}wrist_2_link" />
       <origin xyz="-0.03 0.0 0.231" rpy="0 0 0" />
       <axis xyz="0 0 1" />
@@ -154,5 +154,5 @@
         <origin xyz="0.0 0.0 0.03" rpy="0 0 ${pi}" />
         <geometry>
-      <box size="0.06 0.13 0.09" />
+          <box size="0.06 0.13 0.09" />
         </geometry>
       </collision>
@@ -168,7 +168,7 @@
         <mass value="0.491" />
         <inertia
-        ixx="1.0" ixy="0.0" ixz="0.0"
-        iyy="1.0" iyz="0.0"
-        izz="1.0"/>
+          ixx="1.0" ixy="0.0" ixz="0.0"
+          iyy="1.0" iyz="0.0"
+          izz="1.0"/>
       </inertial>
     </link>
@@ -176,5 +176,5 @@
     <joint name="${prefix_val}wrist_2_joint" type="revolute">
       <parent link="${prefix_val}wrist_2_link" />
-      <child link = "${prefix_val}wrist_3_link" />
+      <child link="${prefix_val}wrist_3_link" />
       <origin xyz="0.0 0.0 0.027" rpy="0 0 0" />
       <axis xyz="0 1 0" />
@@ -187,5 +187,5 @@
         <origin xyz="0.0 0.0 0.08" rpy="0 0 ${pi}" />
         <geometry>
-      <box size="0.07 0.07 0.08" />
+          <box size="0.07 0.07 0.08" />
         </geometry>
       </collision>
@@ -201,7 +201,7 @@
         <mass value="0.454" />
         <inertia
-        ixx="1.0" ixy="0.0" ixz="0.0"
-        iyy="1.0" iyz="0.0"
-        izz="1.0"/>
+          ixx="1.0" ixy="0.0" ixz="0.0"
+          iyy="1.0" iyz="0.0"
+          izz="1.0"/>
       </inertial>
     </link>
@@ -209,5 +209,5 @@
     <joint name="${prefix_val}wrist_3_joint" type="revolute">
       <parent link="${prefix_val}wrist_3_link" />
-      <child link = "${prefix_val}ee_link" />
+      <child link="${prefix_val}ee_link" />
       <origin xyz="0.0 0.0 0.123" rpy="0 0 0" />
       <axis xyz="0 0 1" />
@@ -220,5 +220,5 @@
         <origin xyz="0.0 0.0 0.0" rpy="0 0 0" />
         <geometry>
-          <box size = "0.01 0.01 0.01"/>
+          <box size="0.01 0.01 0.01"/>
         </geometry>
       </collision>
@@ -226,5 +226,5 @@
         <origin xyz="0.0 0.0 0.0" rpy="0 0 0" />
         <geometry>
-          <box size = "0.01 0.01 0.01"/>
+          <box size="0.01 0.01 0.01"/>
         </geometry>
         <material name="red"/>
@@ -234,7 +234,7 @@
         <mass value="0.001" />
         <inertia
-        ixx="1.0" ixy="0.0" ixz="0.0"
-        iyy="1.0" iyz="0.0"
-        izz="1.0"/>
+          ixx="1.0" ixy="0.0" ixz="0.0"
+          iyy="1.0" iyz="0.0"
+          izz="1.0"/>
       </inertial>
     </link>

Commit message: Update the arm collision model

File: manipulator_description/urdf/manipulator_h.xacro (robot description, xacro)
@@ -22,5 +22,5 @@
         <origin xyz="0 0 0.063" rpy="0 0 ${pi}"/>
         <geometry>
-          <box size="0.06 0.06 0.126"/>
+          <box size="0.054 0.054 0.126"/>
         </geometry>
       </collision>
@@ -53,7 +53,7 @@
     <link name="${prefix_val}upper_arm_link">
       <collision>
-        <origin xyz="0 0 0.033" rpy="0 0 ${pi}"/>
-        <geometry>
-          <box size="0.07 0.15 0.08"/>
+        <origin xyz="0 0 0.03" rpy="0 0 ${pi}"/>
+        <geometry>
+          <box size="0.06 0.14 0.06"/>
         </geometry>
       </collision>
@@ -86,7 +86,7 @@
     <link name="${prefix_val}forearm_link">
       <collision>
-        <origin xyz="0.02 0 0.15" rpy="0 0 ${pi}"/>
-        <geometry>
-          <box size="0.1 0.15 0.25"/>
+        <origin xyz="-.001 0 0.148" rpy="${pi/2} 0 ${pi}"/>
+        <geometry>
+          <mesh filename="package://manipulator_description/meshes/collision/link3.stl"/>
         </geometry>
       </collision>
@@ -119,7 +119,7 @@
     <link name="${prefix_val}wrist_1_link">
       <collision>
-        <origin xyz="-0.01 0.0 0.1" rpy="0 0 ${pi}" />
-        <geometry>
-          <box size="0.1 0.15 0.25" />
+        <origin xyz="-0.03 0.0 0.1285" rpy="${pi/2} 0 ${pi}" />
+        <geometry>
+          <mesh filename="package://manipulator_description/meshes/collision/link4.stl"/>
         </geometry>
       </collision>
@@ -152,7 +152,7 @@
     <link name="${prefix_val}wrist_2_link">
       <collision>
-        <origin xyz="0.0 0.0 0.03" rpy="0 0 ${pi}" />
-        <geometry>
-          <box size="0.06 0.13 0.09" />
+        <origin xyz="0.0 0.0 0.024" rpy="0 0 ${pi}" />
+        <geometry>
+          <box size="0.048 0.09 0.048" />
         </geometry>
       </collision>
@@ -185,7 +185,7 @@
     <link name="${prefix_val}wrist_3_link">
       <collision>
-        <origin xyz="0.0 0.0 0.08" rpy="0 0 ${pi}" />
-        <geometry>
-          <box size="0.07 0.07 0.08" />
+        <origin xyz="0.0 0.0 0.081" rpy="${pi/2} 0 ${pi/2}" />
+        <geometry>
+          <mesh filename="package://manipulator_description/meshes/collision/link6.stl"/>
         </geometry>
       </collision>
