Commit message: Modified inertial params

File: manipulator_description/urdf/manipulator_h.xacro (robot description, xacro)
@@ -33,10 +33,10 @@
       </visual>
       <inertial>
-        <origin xyz="0 0 0" rpy="0 0 0"/>
-        <mass value="0.936"/>
-        <inertia
-          ixx="1.0" ixy="0.0" ixz="0.0"
-          iyy="1.0" iyz="0.0"
-          izz="1.0"/>
+        <!-- <origin xyz="0 0 0" rpy="0 0 0"/> -->
+        <!-- <mass value="0.936"/> -->
+        <!-- <inertia ixx="1.0" ixy="0.0" ixz="0.0" iyy="1.0" iyz="0.0" izz="1.0" /> -->
+        <origin xyz="0.00023 0.00000 0.06223" rpy="0 0 0"/>
+        <mass value="0.85644"/>
+        <inertia ixx="0.00121064" ixy="0.0" ixz="0.00001100" iyy="0.00120886" iyz="0.0" izz="0.00038103" />
       </inertial>
     </link>
@@ -48,5 +48,5 @@
       <axis xyz="0 0 1"/>
       <limit velocity="6.5" effort="1000" lower="${-pi*0.95}" upper="${pi*0.95}" />
-      <dynamics damping="0.7"/>
+      <dynamics damping="0"/>
     </joint>
     <!-- link 2 -->
@@ -66,10 +66,10 @@
       </visual>
       <inertial>
-        <origin xyz="0 0 0" rpy="0 0 0"/>
-        <mass value="1.030"/>
-        <inertia
-          ixx="1.0" ixy="0.0" ixz="0.0"
-          iyy="1.0" iyz="0.0"
-          izz="1.0"/>
+        <!-- <origin xyz="0 0 0" rpy="0 0 0"/> -->
+        <!-- <mass value="1.030"/> -->
+        <!-- <inertia ixx="1.0" ixy="0.0" ixz="0.0" iyy="1.0" iyz="0.0" izz="1.0" /> -->
+        <origin xyz="0.00000 0.00080 0.03183" rpy="0 0 0"/>
+        <mass value="0.94658"/>
+        <inertia ixx="0.00152547" ixy="0.0" ixz="0.0" iyy="0.00045954" iyz="-0.00001086" izz="0.00151740" />
       </inertial>
     </link>
@@ -81,5 +81,5 @@
       <axis xyz="0 1 0"/>
       <limit velocity="6.5" effort="1000" lower="${-pi*0.6}" upper="${pi*0.6}" />
-      <dynamics damping="0.7"/>
+      <dynamics damping="0"/>
     </joint>
     <!-- link 3 -->
@@ -99,10 +99,9 @@
       </visual>
       <inertial>
-        <origin xyz="0 0 0" rpy="0 0 0"/>
-        <mass value="1.404"/>
-        <inertia
-          ixx="1.0" ixy="0.0" ixz="0.0"
-          iyy="1.0" iyz="0.0"
-          izz="1.0"/>
+        <origin xyz="0 0 0.148" rpy="0 0 0"/>
+        <!-- <mass value="1.404"/> -->
+        <!-- <inertia ixx="1.0" ixy="0.0" ixz="0.0" iyy="1.0" iyz="0.0" izz="1.0" /> -->
+        <mass value="1.30260"/>
+        <inertia ixx="0.01111021" ixy="0.00001331" ixz="-0.00134208" iyy="0.01046642" iyz="0.00016235" izz="0.00202081" />
       </inertial>
     </link>
@@ -114,5 +113,5 @@
       <axis xyz="0 1 0"/>
       <limit velocity="6.5" effort="1000" lower="${-pi*0.4}" upper="${pi*0.72}" />
-      <dynamics damping="0.7"/>
+      <dynamics damping="0"/>
     </joint>
     <!-- link 4 -->
@@ -132,10 +131,9 @@
       </visual>
       <inertial>
-        <origin xyz="0 0 0" rpy="0 0 0" />
-        <mass value="1.236" />
-        <inertia
-          ixx="1.0" ixy="0.0" ixz="0.0"
-          iyy="1.0" iyz="0.0"
-          izz="1.0"/>
+        <origin xyz="-0.03 0 0.1285" rpy="0 ${pi/2} 0" />
+        <!-- <mass value="1.236" /> -->
+        <!-- <inertia ixx="1.0" ixy="0.0" ixz="0.0" iyy="1.0" iyz="0.0" izz="1.0" /> -->
+        <mass value="1.15977"/>
+        <inertia ixx="0.00096726" ixy="0.00004383" ixz="-0.00002771" iyy="0.00318801" iyz="0.00000627" izz="0.00341484" />
       </inertial>
     </link>
@@ -147,5 +145,5 @@
       <axis xyz="0 0 1" />
       <limit velocity="6.5" effort="1000" lower="${-pi}" upper="${pi}" />
-      <dynamics damping="0.7"/>
+      <dynamics damping="0"/>
     </joint>
     <!-- link 5 -->
@@ -165,10 +163,9 @@
       </visual>
       <inertial>
-        <origin xyz="0 0 0" rpy="0 0 0" />
-        <mass value="0.491" />
-        <inertia
-          ixx="1.0" ixy="0.0" ixz="0.0"
-          iyy="1.0" iyz="0.0"
-          izz="1.0"/>
+        <origin xyz="0 0 0.024" rpy="0 0 0" />
+        <!-- <mass value="0.491" /> -->
+        <!-- <inertia ixx="1.0" ixy="0.0" ixz="0.0" iyy="1.0" iyz="0.0" izz="1.0" /> -->
+        <mass value="0.44688"/>
+        <inertia ixx="0.00030285" ixy="0.00000761" ixz="0.00000031" iyy="0.00022339" iyz="-0.00000001" izz="0.00039766" />
       </inertial>
     </link>
@@ -180,5 +177,5 @@
       <axis xyz="0 1 0" />
       <limit velocity="6.5" effort="1000" lower="${-pi*0.5}" upper="${pi*0.5}" />
-      <dynamics damping="0.7"/>
+      <dynamics damping="0"/>
     </joint>
     <!-- link 6 -->
@@ -198,10 +195,9 @@
       </visual>
       <inertial>
-        <origin xyz="0 0 0" rpy="0 0 0" />
-        <mass value="0.454" />
-        <inertia
-          ixx="1.0" ixy="0.0" ixz="0.0"
-          iyy="1.0" iyz="0.0"
-          izz="1.0"/>
+        <origin xyz="0 0 0.081" rpy="${pi/2} ${pi/2} 0" />
+        <!-- <mass value="0.454" /> -->
+        <!-- <inertia ixx="1.0" ixy="0.0" ixz="0.0" iyy="1.0" iyz="0.0" izz="1.0" /> -->
+        <mass value="0.43273"/>
+        <inertia ixx="0.00021512" ixy="0.00001009" ixz="0.00000000" iyy="0.00042827" iyz="0.00000000" izz="0.00051436" />
       </inertial>
     </link>
@@ -213,5 +209,5 @@
       <axis xyz="0 0 1" />
       <limit velocity="6.5" effort="1000" lower="${-pi}" upper="${pi}" />
-      <dynamics damping="0.7"/>
+      <dynamics damping="0"/>
     </joint>
     <!-- End Effector -->
@@ -231,10 +227,9 @@
       </visual>
       <inertial>
-        <origin xyz="0.0 0.0 0.0" rpy="0 0 0" />
-        <mass value="0.001" />
-        <inertia
-          ixx="1.0" ixy="0.0" ixz="0.0"
-          iyy="1.0" iyz="0.0"
-          izz="1.0"/>
+        <origin xyz="0 0 0" rpy="0 0 0"/>
+        <!-- <mass value="0.001" /> -->
+        <!-- <inertia ixx="1.0" ixy="0.0" ixz="0.0" iyy="1.0" iyz="0.0" izz="1.0" /> -->
+        <mass value="0.01919"/>
+        <inertia ixx="0.00000938" ixy="0.0" ixz="0.0" iyy="0.00000338" iyz="0.0" izz="0.00000635" />
       </inertial>
     </link>
