Commit message: Clean up file into a macro

File: manipulator_description/urdf/common.xacro (robot description, xacro)
@@ -1,23 +1,12 @@
 <?xml version="1.0"?>
 <robot xmlns:xacro="http://www.ros.org/wiki/xacro">
-  <gazebo>
-    <plugin name="ros_control" filename="libgazebo_ros_control.so">
-      <!--robotNamespace>/</robotNamespace-->
-      <!--robotSimType>gazebo_ros_control/DefaultRobotHWSim</robotSimType-->
-    </plugin>
-<!--
-    <plugin name="gazebo_ros_power_monitor_controller" filename="libgazebo_ros_power_monitor.so">
-      <alwaysOn>true</alwaysOn>
-      <updateRate>1.0</updateRate>
-      <timeout>5</timeout>
-      <powerStateTopic>power_state</powerStateTopic>
-      <powerStateRate>10.0</powerStateRate>
-      <fullChargeCapacity>87.78</fullChargeCapacity>
-      <dischargeRate>-474</dischargeRate>
-      <chargeRate>525</chargeRate>
-      <dischargeVoltage>15.52</dischargeVoltage>
-      <chargeVoltage>16.41</chargeVoltage>
-    </plugin>
--->
-  </gazebo>
+  <!-- ros_control plugin -->
+  <xacro:macro name="manipulator_arm_gazebo" params="prefix prefix_val">
+    <gazebo>
+      <plugin name="${prefix_val}ros_control" filename="libgazebo_ros_control.so">
+        <robotNamespace>${prefix}</robotNamespace>
+        <!--robotSimType>gazebo_ros_control/DefaultRobotHWSim</robotSimType-->
+      </plugin>
+    </gazebo>
+  </xacro:macro>
 </robot>

Commit message: Add prefix_val generation from prefix to common

File: manipulator_description/urdf/common.xacro (robot description, xacro)
@@ -1,6 +1,11 @@
 <?xml version="1.0"?>
 <robot xmlns:xacro="http://www.ros.org/wiki/xacro">
+  <xacro:property name="prefix_val" value="" />
   <!-- ros_control plugin -->
-  <xacro:macro name="manipulator_arm_gazebo" params="prefix prefix_val">
+  <xacro:macro name="manipulator_arm_gazebo" params="prefix">
+    <!-- Suffix prefix with underscore -->
+    <xacro:if value="${prefix.__len__()}">
+      <xacro:property name="prefix_val" value="${prefix + '_'}" />
+    </xacro:if>
     <gazebo>
       <plugin name="${prefix_val}ros_control" filename="libgazebo_ros_control.so">

Commit message: Fix inertia

File: manipulator_description/urdf/common.xacro (robot description, xacro)
@@ -13,5 +13,5 @@
         <robotNamespace>${prefix}</robotNamespace>
         <filterJointsParam>joint_names</filterJointsParam>
-        <!--robotSimType>gazebo_ros_control/DefaultRobotHWSim</robotSimType-->
+        <robotSimType>gazebo_ros_control/DefaultRobotHWSim</robotSimType>
       </plugin>
     </gazebo>

File: manipulator_description/urdf/manipulator_h.xacro (robot description, xacro)
@@ -6,5 +6,5 @@
   <xacro:property name="pi" value="3.141592654" />
   <xacro:property name="prefix_val" value="" />
-  <xacro:macro name="manipulator_h_arm" params="prefix joint_limited parent *origin">
+  <xacro:macro name="manipulator_h_arm" params="prefix joint_limited parent dummy_ee_link:=false *origin">
     <!-- Suffix prefix with underscore -->
     <xacro:if value="${prefix.__len__()}">
@@ -38,5 +38,6 @@
         <origin xyz="0.00023 0.00000 0.06223" rpy="0 0 0"/>
         <mass value="0.85644"/>
-        <inertia ixx="0.00121064" ixy="0.0" ixz="0.00001100" iyy="0.00120886" iyz="0.0" izz="0.00038103" />
+        <!-- <inertia ixx="0.00121064" ixy="0.0" ixz="0.00001100" iyy="0.00120886" iyz="0.0" izz="0.00038103" /> -->
+        <inertia ixx="0.00134118504" ixy="0.0" ixz="0.0" iyy="0.00134118504" iyz="0.0" izz="0.00041622984" />
       </inertial>
     </link>
@@ -71,5 +72,6 @@
         <origin xyz="0.00000 0.00080 0.03183" rpy="0 0 0"/>
         <mass value="0.94658"/>
-        <inertia ixx="0.00152547" ixy="0.0" ixz="0.0" iyy="0.00045954" iyz="-0.00001086" izz="0.00151740" />
+        <!-- <inertia ixx="0.00152547" ixy="0.0" ixz="0.0" iyy="0.00045954" iyz="-0.00001086" izz="0.00151740" /> -->
+        <inertia ixx="0.00183005466667" ixy="0.0" ixz="0.0" iyy="0.000567948" iyz="0.0" izz="0.00183005466667" />
       </inertial>
     </link>
@@ -103,5 +105,6 @@
         <!-- <inertia ixx="1.0" ixy="0.0" ixz="0.0" iyy="1.0" iyz="0.0" izz="1.0" /> -->
         <mass value="1.30260"/>
-        <inertia ixx="0.01111021" ixy="0.00001331" ixz="-0.00134208" iyy="0.01046642" iyz="0.00016235" izz="0.00202081" />
+        <!-- <inertia ixx="0.01111021" ixy="0.00001331" ixz="-0.00134208" iyy="0.01046642" iyz="0.00016235" izz="0.00202081" /> -->
+        <inertia ixx="0.0136625102365" ixy="0.0" ixz="0.0" iyy="0.0124082569044" iyz="0.0" izz="0.00324753226791" />
       </inertial>
     </link>
@@ -135,5 +138,6 @@
         <!-- <inertia ixx="1.0" ixy="0.0" ixz="0.0" iyy="1.0" iyz="0.0" izz="1.0" /> -->
         <mass value="1.15977"/>
-        <inertia ixx="0.00096726" ixy="0.00004383" ixz="-0.00002771" iyy="0.00318801" iyz="0.00000627" izz="0.00341484" />
+        <!-- <inertia ixx="0.00096726" ixy="0.00004383" ixz="-0.00002771" iyy="0.00318801" iyz="0.00000627" izz="0.00341484" /> -->
+        <inertia ixx="0.00205032491251" ixy="0.0" ixz="0.0" iyy="0.00691847164616" iyz="0.0" izz="0.00765159473365" />
       </inertial>
     </link>
@@ -167,5 +171,6 @@
         <!-- <inertia ixx="1.0" ixy="0.0" ixz="0.0" iyy="1.0" iyz="0.0" izz="1.0" /> -->
         <mass value="0.44688"/>
-        <inertia ixx="0.00030285" ixy="0.00000761" ixz="0.00000031" iyy="0.00022339" iyz="-0.00000001" izz="0.00039766" />
+        <!-- <inertia ixx="0.00030285" ixy="0.00000761" ixz="0.00000031" iyy="0.00022339" iyz="-0.00000001" izz="0.00039766" /> -->
+        <inertia ixx="0.00038744496" ixy="0.0" ixz="0.0" iyy="0.00017160192" iyz="0.0" izz="0.00038744496" />
       </inertial>
     </link>
@@ -199,5 +204,6 @@
         <!-- <inertia ixx="1.0" ixy="0.0" ixz="0.0" iyy="1.0" iyz="0.0" izz="1.0" /> -->
         <mass value="0.43273"/>
-        <inertia ixx="0.00021512" ixy="0.00001009" ixz="0.00000000" iyy="0.00042827" iyz="0.00000000" izz="0.00051436" />
+        <!-- <inertia ixx="0.00021512" ixy="0.00001009" ixz="0.00000000" iyy="0.00042827" iyz="0.00000000" izz="0.00051436" /> -->
+        <inertia ixx="0.00039594795" ixy="0.0" ixz="0.0" iyy="0.00104401581334" iyz="0.0" izz="0.000775290483338" />
       </inertial>
     </link>
@@ -213,24 +219,33 @@
     <!-- End Effector -->
     <link name="${prefix_val}ee_link">
-      <collision>
-        <origin xyz="0.0 0.0 0.0" rpy="0 0 0" />
-        <geometry>
-          <box size="0.01 0.01 0.01"/>
-        </geometry>
-      </collision>
-      <visual>
-        <origin xyz="0.0 0.0 0.0" rpy="0 0 0" />
-        <geometry>
-          <box size="0.01 0.01 0.01"/>
-        </geometry>
-        <material name="red"/>
-      </visual>
-      <inertial>
-        <origin xyz="0 0 0" rpy="0 0 0"/>
-        <!-- <mass value="0.001" /> -->
-        <!-- <inertia ixx="1.0" ixy="0.0" ixz="0.0" iyy="1.0" iyz="0.0" izz="1.0" /> -->
-        <mass value="0.01919"/>
-        <inertia ixx="0.00000938" ixy="0.0" ixz="0.0" iyy="0.00000338" iyz="0.0" izz="0.00000635" />
-      </inertial>
+      <xacro:unless value="${dummy_ee_link}">
+        <collision>
+          <origin xyz="0.0 0.0 0.025" rpy="0 0 0" />
+          <geometry>
+            <box size="0.05 0.05 0.05"/>
+          </geometry>
+        </collision>
+        <visual>
+          <origin xyz="0.0 0.0 0.025" rpy="0 0 0" />
+          <geometry>
+            <box size="0.05 0.05 0.05"/>
+          </geometry>
+          <material name="red"/>
+        </visual>
+        <inertial>
+          <origin xyz="0 0 0" rpy="0 0 0"/>
+          <mass value="0.1" />
+          <inertia ixx="0.0000416666666667" ixy="0.0" ixz="0.0" iyy="0.0000416666666667" iyz="0.0" izz="0.0000416666666667" />
+        </inertial>
+          <!-- <inertia ixx="0.0000016666" ixy="0.0" ixz="0.0" iyy="0.0000016666" iyz="0.0" izz="0.0000016666" /> -->
+        <!-- <inertial>
+          <origin xyz="0 0 0" rpy="0 0 0"/> -->
+          <!-- <mass value="0.001" /> -->
+          <!-- <inertia ixx="1.0" ixy="0.0" ixz="0.0" iyy="1.0" iyz="0.0" izz="1.0" /> -->
+          <!-- <mass value="0.01919"/> -->
+          <!-- <inertia ixx="0.00000938" ixy="0.0" ixz="0.0" iyy="0.00000338" iyz="0.0" izz="0.00000635" /> -->
+          <!-- <inertia ixx="0.0000011983" ixy="0.0" ixz="0.0" iyy="0.0000011983" iyz="0.0" izz="0.0000011983" />
+        </inertial> -->
+      </xacro:unless>
     </link>
     <xacro:manipulator_arm_transmission prefix="${prefix_val}" />
