Commit message: Dont know what this change means

File: manipulator_description/urdf/manipulator_h_arm.xacro (robot description, xacro)
@@ -10,5 +10,5 @@
   <!-- arm -->
   <xacro:manipulator_h_arm prefix="" parent="world" joint_limited="false">
-    <origin xyz="0 0 0" rpy="0 0 0" />
+    <origin xyz="0 0 1" rpy="0 1.5707963267948966 0 " />
   </xacro:manipulator_h_arm>
 </robot>
